Commit message: add ros2_control

File: pal_gripper_description/urdf/gripper.ros2_control.xacro (robot description, xacro)
@@ -20,6 +20,20 @@
       <state_interface name="effort" />
     </joint>
+    <joint name="${name}_right_finger_joint">
+      <command_interface name="position" />
+      <state_interface name="position" />
+      <state_interface name="velocity" />
+      <state_interface name="effort" />
+    </joint>
+    <joint name="${name}_left_finger_joint">
+      <command_interface name="position" />
+      <state_interface name="position" />
+      <state_interface name="velocity" />
+      <state_interface name="effort" />
+    </joint>
     <xacro:include filename="$(find pal_gripper_description)/urdf/gripper.transmission.xacro" />
     <xacro:gripper_simple_transmission name="${name}" reduction="${reduction}" />
+    <xacro:gripper_simple_transmission name="${name}_right_finger" reduction="${reduction}" />
+    <xacro:gripper_simple_transmission name="${name}_left_finger" reduction="${reduction}" />
   </xacro:macro>
 </robot>
