Commit message: changed inertia
Signed-off-by: Juancams <jc.manzanares.serrano@gmail.com>

File: pal_gripper_description/urdf/gripper.urdf.xacro (robot description, xacro)
@@ -56,7 +56,7 @@
       <origin rpy="0 0 0" xyz="-0.004470 0.010766 -0.121013" />
       <mass value="0.109980" />
-      <!-- <inertia ixx="0.000232" ixy="0.000005" ixz="0.000032"
-               iyy="0.000224" iyz="0.000036"
-               izz="0.000029" /> -->
+      <inertia ixx="0.0" ixy="0.0" ixz="0.0"
+               iyy="0.0" iyz="0.0"
+               izz="0.0" />
     </inertial>
     <visual>
@@ -94,7 +94,7 @@
       <origin rpy="0 0 0" xyz="-0.004470 0.010766 -0.121013" />
       <mass value="0.109980" />
-      <!-- <inertia ixx="0.000232" ixy="0.000005" ixz="0.000032"
-               iyy="0.000224" iyz="0.000036"
-               izz="0.000029" /> -->
+      <inertia ixx="0.0" ixy="0.0" ixz="0.0"
+               iyy="0.0" iyz="0.0"
+               izz="0.0" />
     </inertial>
     <visual>

Commit message: Solved error with joint limit

File: pal_gripper_description/urdf/gripper.urdf.xacro (robot description, xacro)
@@ -82,10 +82,10 @@
     <child link="${name}_right_finger_link" />
     <axis xyz="1 0 0" />
-    <limit effort="16" lower="0.0" upper="0.045" velocity="0.05" />
+    <limit effort="16" lower="-0.001" upper="0.045" velocity="0.05" />
     <calibration rising="0.0" />
     <dynamics damping="80" friction="2.0"/>
     <safety_controller k_position="20"
                        k_velocity="20"
-                       soft_lower_limit="${0.0 + gripper_eps}"
+                       soft_lower_limit="${0.0 - gripper_eps}"
                        soft_upper_limit="${0.045 - gripper_eps}" />
   </joint>
@@ -120,10 +120,10 @@
     <child link="${name}_left_finger_link" />
     <axis xyz="-1 0 0" />
-    <limit effort="16" lower="0" upper="0.045" velocity="0.05" />
+    <limit effort="16" lower="-0.001" upper="0.045" velocity="0.05" />
     <calibration rising="0.0" />
     <dynamics damping="80" friction="2.0"/>
     <safety_controller k_position="20"
                        k_velocity="20"
-                       soft_lower_limit="${0.0 + gripper_eps}"
+                       soft_lower_limit="${0.0 - gripper_eps}"
                        soft_upper_limit="${0.045 - gripper_eps}" />
   </joint>
