Commit message: add fixed link

File: pal_gripper_description/robots/gripper_test.urdf.xacro (robot description, xacro)
@@ -19,9 +19,18 @@
   <xacro:include filename="$(find pal_urdf_utils)/urdf/materials.urdf.xacro" />
   <!-- Generic simulator_gazebo plugins -->
+  <!-- ros2_control -->
+  <xacro:include filename="$(find pal_gripper_description)/ros2_control/ros2_control.urdf.xacro" />
+  <xacro:pal_gripper_ros2_control use_sim_time="$(arg use_sim_time)" />
   <xacro:include filename="$(find pal_gripper_description)/gazebo/gazebo.urdf.xacro" />
+    <link name="world"/>
+    <joint name="world_fixed" type="fixed">
+        <origin xyz="0 0 0.1" rpy="0 0 0"/>
+        <parent link="world"/>
+        <child link="base_link"/>
+    </joint>
   <!--Spawn gripper-->
   <link name="base_link"/>
   <xacro:pal_gripper parent="base_link" name="gripper">
-    <origin xyz="0 0 0" rpy="0 ${180 * deg_to_rad} ${0 * deg_to_rad}" />
+    <origin xyz="0 0 0" rpy="${0 * deg_to_rad} ${-180 * deg_to_rad} 0" />
   </xacro:pal_gripper>
 </robot>
