Commit message: follow gripper ros2 structure

File: pal_gripper_description/ros2_control/ros2_control.urdf.xacro (robot description, xacro)
@@ -26,5 +26,6 @@
       </hardware>
       <!-- pal-gripper -->
-      <xacro:ros2_control_gripper name="gripper" reduction="1.0" />
+      <xacro:ros2_control_gripper name="gripper_left_finger" reduction="1.0" />
+      <xacro:ros2_control_gripper name="gripper_right_finger" reduction="1.0" />
     </ros2_control>
   </xacro:macro>

File: pal_gripper_description/urdf/gripper.ros2_control.xacro (robot description, xacro)
@@ -20,20 +20,6 @@
       <state_interface name="effort" />
     </joint>
-    <joint name="${name}_right_finger_joint">
-      <command_interface name="position" />
-      <state_interface name="position" />
-      <state_interface name="velocity" />
-      <state_interface name="effort" />
-    </joint>
-    <joint name="${name}_left_finger_joint">
-      <command_interface name="position" />
-      <state_interface name="position" />
-      <state_interface name="velocity" />
-      <state_interface name="effort" />
-    </joint>
     <xacro:include filename="$(find pal_gripper_description)/urdf/gripper.transmission.xacro" />
     <xacro:gripper_simple_transmission name="${name}" reduction="${reduction}" />
-    <xacro:gripper_simple_transmission name="${name}_right_finger" reduction="${reduction}" />
-    <xacro:gripper_simple_transmission name="${name}_left_finger" reduction="${reduction}" />
   </xacro:macro>
 </robot>
