Commit message: Harmonic
Signed-off-by: Juancams <jc.manzanares.serrano@gmail.com>

File: pal_gripper_description/gazebo/gazebo.urdf.xacro (robot description, xacro)
@@ -14,5 +14,5 @@
 <robot xmlns:xacro="http://ros.org/wiki/xacro" name="pal_gripper">
     <gazebo>
-      <plugin filename="libgazebo_ros2_control.so" name="gazebo_ros2_control">
+      <plugin filename="libgz_ros2_control-system.so" name="gz_ros2_control::GazeboSimROS2ControlPlugin">
         <parameters>$(find pal_gripper_controller_configuration)/config/gazebo_controller_manager_cfg.yaml</parameters>
       </plugin>

File: pal_gripper_description/ros2_control/ros2_control.urdf.xacro (robot description, xacro)
@@ -19,5 +19,5 @@
       <hardware>
         <xacro:if value="$(arg use_sim_time)">
-          <plugin>gazebo_ros2_control/GazeboSystem</plugin>
+          <plugin>gz_ros2_control/GazeboSimSystem</plugin>
         </xacro:if>
         <xacro:unless value="$(arg use_sim_time)">

File: pal_gripper_description/urdf/gripper.urdf.xacro (robot description, xacro)
@@ -32,5 +32,5 @@
       <origin rpy="0 0 0" xyz="0 0 0" />
       <geometry>
-        <mesh filename="package://pal_gripper_description/meshes/gripper_link.stl"/>
+        <mesh filename="file://$(find pal_gripper_description)/meshes/gripper_link.stl"/>
       </geometry>
       <material name="White"/>
@@ -39,5 +39,5 @@
       <origin rpy="0 0 0" xyz="0 0 0" />
       <geometry>
-        <mesh filename="package://pal_gripper_description/meshes/gripper_link_collision.stl"/>
+        <mesh filename="file://$(find pal_gripper_description)/meshes/gripper_link_collision.stl"/>
       </geometry>
     </collision>
@@ -56,12 +56,12 @@
       <origin rpy="0 0 0" xyz="-0.004470 0.010766 -0.121013" />
       <mass value="0.109980" />
-      <inertia ixx="0.000232" ixy="-0.000005" ixz="-0.000032"
+      <!-- <inertia ixx="0.000232" ixy="0.000005" ixz="0.000032"
                iyy="0.000224" iyz="0.000036"
-               izz="0.000029" />
+               izz="0.000029" /> -->
     </inertial>
     <visual>
       <origin rpy="0 0 3.1415" xyz="0 0 0" />
       <geometry>
-        <mesh filename="package://pal_gripper_description/meshes/gripper_finger_link.stl" scale="-1 -1 1"/>
+        <mesh filename="file://$(find pal_gripper_description)/meshes/gripper_finger_link.stl" scale="-1 -1 1"/>
       </geometry>
       <material name="Black"/>
@@ -94,12 +94,12 @@
       <origin rpy="0 0 0" xyz="-0.004470 0.010766 -0.121013" />
       <mass value="0.109980" />
-      <inertia ixx="0.000232" ixy="-0.000005" ixz="-0.000032"
+      <!-- <inertia ixx="0.000232" ixy="0.000005" ixz="0.000032"
                iyy="0.000224" iyz="0.000036"
-               izz="0.000029" />
+               izz="0.000029" /> -->
     </inertial>
     <visual>
       <origin rpy="0 0 3.1415" xyz="0 0 0"/>
       <geometry>
-        <mesh filename="package://pal_gripper_description/meshes/gripper_finger_link.stl"/>
+        <mesh filename="file://$(find pal_gripper_description)/meshes/gripper_finger_link.stl"/>
       </geometry>
       <material name="Black"/>
